Commit message: added the kinematics for the robot with the end effector

File: src/arduinobot_description/src/urdf/arduinobot.urdf (robot description, URDF)
Before this commit: robot arduinobot, 7 links, 6 joints
Links:
- added link gripper_left, mass 0.1; collision mesh filename=package://arduinobot_description/src/mesh/left_finger.STL scale=0.01 0.01 0.01; visual mesh filename=package://arduinobot_description/src/mesh/left_finger.STL scale=0.01 0.01 0.01
- added link gripper_right, mass 0.1; collision mesh filename=package://arduinobot_description/src/mesh/right_finger.STL scale=0.01 0.01 0.01; visual mesh filename=package://arduinobot_description/src/mesh/right_finger.STL scale=0.01 0.01 0.01
- link base_link: mass None -> 0.1; geometry collision mesh filename=package://arduinobot_description/src/mesh/basement.STL scale=0.01 0.01 0.01; visual mesh filename=package://arduinobot_description/src/mesh/basement.STL scale=0.01 0.01 0.01
- link base_plate: mass None -> 0.1; geometry collision mesh filename=package://arduinobot_description/src/mesh/round_plate.STL scale=0.01 0.01 0.01; visual mesh filename=package://arduinobot_description/src/mesh/base_plate.STL scale=0.01 0.01 0.01
- link claw_support: mass None -> 0.1; geometry collision mesh filename=package://arduinobot_description/src/mesh/claw_support.STL scale=0.01 0.01 0.01; visual mesh filename=package://arduinobot_description/src/mesh/claw_support.STL scale=0.01 0.01 0.01
- link forward_drive_arm: mass None -> 0.1; geometry collision mesh filename=package://arduinobot_description/src/mesh/forward_drive_arm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 scale=0.01 0.01 0.01; visual mesh filename=package://arduinobot_description/src/mesh/forward_drive_arm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 scale=0.01 0.01 0.01
- link horizontal_arm: mass None -> 0.1; geometry collision mesh filename=package://arduinobot_description/src/mesh/horizontal_arm.STL scale=0.01 0.01 0.01; visual mesh filename=package://arduinobot_description/src/mesh/horizontal_arm.STL scale=0.01 0.01 0.01
Joints:
- removed joint claw_support_to_tool
- added joint gripper_right_to_tool: type fixed, parent gripper_right, child tool_link, origin xyz=0 0 0
- added joint joint_4: type revolute, parent claw_support, child gripper_right, origin xyz=-0.04 0.13 -0.1, axis 0 0 1, limit lower=-1.5707963268 upper=0 effort=1000.0 velocity=0.5
- added joint joint_5: type revolute, parent claw_support, child gripper_left, origin xyz=-0.22 0.13 -0.1, axis 0 0 1, limit lower=0 upper=1.5707963268 effort=1000.0 velocity=0.5, mimic joint=joint_4 multiplier=-1 offset=0
