Commit message: clean the urdf file with xacro

File: arduinobot_ws/src/arduinobot_description/urdf/arduinobot.urdf (robot description, URDF)
Before this commit: robot arduinobot, 9 links, 8 joints
Joints:
- joint joint_1: limit lower=-1.5707963268 upper=1.5707963268 effort=30.0 velocity=0.5 -> lower=-1.5707963268 upper=1.5707963268 effort=30 velocity=0.5
- joint joint_2: limit lower=-1.5707963268 upper=1.5707963268 effort=30.0 velocity=0.5 -> lower=-1.5707963268 upper=1.5707963268 effort=30 velocity=0.5
- joint joint_3: limit lower=-1.5707963268 upper=1.5707963268 effort=30.0 velocity=0.5 -> lower=-1.5707963268 upper=1.5707963268 effort=30 velocity=0.5
- joint joint_4: limit lower=-1.5707963268 upper=0 effort=30.0 velocity=0.5 -> lower=-1.5707963268 upper=0 effort=30 velocity=0.5
- joint joint_5: limit lower=0 upper=1.5707963268 effort=30.0 velocity=0.5 -> lower=0 upper=1.5707963268 effort=30 velocity=0.5

File: arduinobot_ws/src/arduinobot_description/urdf/arduinobot.urdf.xacro (robot description, xacro)
@@ -3,4 +3,27 @@
     <!-- Useful Variables (Properties) -->
     <xacro:property name="PI" value="3.14159265359" />
+    <xacro:property name="effort" value="30" />
+    <xacro:property name="velocity" value="0.5" />
+    <!-- Useful Macros -->
+    <xacro:macro name="default_inertial" params="mass">
+        <inertial>
+            <mass value="${mass}" />
+            <inertia ixx="1.0" ixy="0.0" ixz="0.0"
+                     iyy="1.0" iyz="0.0"
+                     izz="1.0" />
+        </inertial>
+    </xacro:macro>
+    <xacro:macro name="default_transmission" params="number">
+        <transmission name="transmission_${number}">
+            <type>transmission_interface/SimpleTransmission</type>
+            <joint name="joint_${number}">
+                <hardwareInterface>hardware_interface/PositionJointInterface</hardwareInterface>
+            </joint>
+            <actuator name="motor_${number}">
+                <hardwareInterface>hardware_interface/PositionJointInterface</hardwareInterface>
+                <mechanicalReduction>1</mechanicalReduction>
+            </actuator>
+        </transmission>
+    </xacro:macro>
     <!-- Links -->
     <link name="world"/>
@@ -11,10 +34,5 @@
     </joint>
     <link name="base_link">
-        <inertial>
-                <mass value="1" />
-                <inertia ixx="1.0" ixy="0.0" ixz="0.0"
-                     iyy="1.0" iyz="0.0"
-                     izz="1.0" />
-        </inertial>
+        <xacro:default_inertial mass="1"/>
         <visual>
             <origin rpy="0 0 0" xyz="-0.5 -0.5 0"/>
@@ -31,10 +49,5 @@
     </link>
     <link name="base_plate">
-        <inertial>
-                <mass value="0.1" />
-                <inertia ixx="1.0" ixy="0.0" ixz="0.0"
-                     iyy="1.0" iyz="0.0"
-                     izz="1.0" />
-        </inertial>
+        <xacro:default_inertial mass="0.1"/>
         <visual>
             <origin rpy="0 0 0" xyz="-0.39 -0.39 -0.56"/>
@@ -51,10 +64,5 @@
     </link>
     <link name="forward_drive_arm">
-        <inertial>
-                <mass value="0.1" />
-                <inertia ixx="1.0" ixy="0.0" ixz="0.0"
-                     iyy="1.0" iyz="0.0"
-                     izz="1.0" />
-        </inertial>
+        <xacro:default_inertial mass="0.1"/>
         <visual>
             <origin rpy=" 0 -${PI/2} ${PI/2}" xyz="0.19 0.06 -0.08"/>
@@ -71,10 +79,5 @@
     </link>
     <link name="horizontal_arm">
-        <inertial>
-                <mass value="0.1" />
-                <inertia ixx="1.0" ixy="0.0" ixz="0.0"
-                     iyy="1.0" iyz="0.0"
-                     izz="1.0" />
-        </inertial>
+        <xacro:default_inertial mass="0.1"/>
         <visual>
             <origin rpy="${PI/2} 0 ${PI/2}" xyz="-0.03 -0.4 -0.06"/>
@@ -91,10 +94,5 @@
     </link>
     <link name="claw_support">
-        <inertial>
-                <mass value="0.05" />
-                <inertia ixx="1.0" ixy="0.0" ixz="0.0"
-                     iyy="1.0" iyz="0.0"
-                     izz="1.0" />
-        </inertial>
+        <xacro:default_inertial mass="0.05"/>
         <visual>
             <origin rpy="0 0 ${PI/2}" xyz="0 -0.05 -0.15"/>
@@ -111,10 +109,5 @@
     </link>
     <link name="gripper_right">
-        <inertial>
-                <mass value="0.01" />
-                <inertia ixx="1.0" ixy="0.0" ixz="0.0"
-                     iyy="1.0" iyz="0.0"
-                     izz="1.0" />
-        </inertial>
+        <xacro:default_inertial mass="0.01"/>
         <visual>
             <origin rpy="0 0 -${PI/2}" xyz="-0.1 0.50 -0.1"/>
@@ -131,10 +124,5 @@
     </link>
     <link name="gripper_left">
-        <inertial>
-                <mass value="0.01" />
-                <inertia ixx="1.0" ixy="0.0" ixz="0.0"
-                     iyy="1.0" iyz="0.0"
-                     izz="1.0" />
-        </inertial>
+        <xacro:default_inertial mass="0.01"/>
         <visual>
             <origin rpy="0 0 -${PI/2}" xyz="-0.04 0.50 -0.1"/>
@@ -157,5 +145,5 @@
         <origin xyz="0 0 0.307"/>
         <axis xyz="0 0 1"/>
-        <limit lower="-${PI/2}" upper="${PI/2}" effort="30.0" velocity="0.5"/>
+        <limit lower="-${PI/2}" upper="${PI/2}" effort="${effort}" velocity="${velocity}"/>
     </joint>
     <joint name ="joint_2" type="revolute">
@@ -164,5 +152,5 @@
         <origin xyz="-0.02 0 0.35"/>
         <axis xyz="1 0 0"/>
-        <limit lower="-${PI/2}" upper="${PI/2}" effort="30.0" velocity="0.5"/>
+        <limit lower="-${PI/2}" upper="${PI/2}" effort="${effort}" velocity="${velocity}"/>
     </joint>
     <joint name ="joint_3" type="revolute">
@@ -171,5 +159,5 @@
         <origin xyz="0 0 0.8"/>
         <axis xyz="1 0 0"/>
-        <limit lower="-${PI/2}" upper="${PI/2}" effort="30.0" velocity="0.5"/>
+        <limit lower="-${PI/2}" upper="${PI/2}" effort="${effort}" velocity="${velocity}"/>
     </joint>
     <joint name ="horizontal_arm_to_claw_support" type="fixed">
@@ -183,5 +171,5 @@
         <origin xyz="-0.04 0.13 -0.1"/>
         <axis xyz="0 0 1"/>
-        <limit lower="-${PI/2}" upper="0" effort="30.0" velocity="0.5"/>
+        <limit lower="-${PI/2}" upper="0" effort="${effort}" velocity="${velocity}"/>
     </joint>
     <joint name ="joint_5" type="revolute">
@@ -190,5 +178,5 @@
         <origin xyz="-0.22 0.13 -0.1"/>
         <axis xyz="0 0 1"/>
-        <limit lower="0" upper="${PI/2}" effort="30.0" velocity="0.5"/>
+        <limit lower="0" upper="${PI/2}" effort="${effort}" velocity="${velocity}"/>
         <mimic joint="joint_4" multiplier="-1" offset="0"/>
     </joint>
@@ -199,55 +187,10 @@
     </joint>
     <!-- Transmissions-->
-    <transmission name="transmission_1">
-        <type>transmission_interface/SimpleTransmission</type>
-        <joint name="joint_1">
-            <hardwareInterface>hardware_interface/PositionJointInterface</hardwareInterface>
-        </joint>
-        <actuator name="motor_1">
-            <hardwareInterface>hardware_interface/PositionJointInterface</hardwareInterface>
-            <mechanicalReduction>1</mechanicalReduction>
-        </actuator>
-    </transmission>
-    <transmission name="transmission_2">
-        <type>transmission_interface/SimpleTransmission</type>
-        <joint name="joint_2">
-            <hardwareInterface>hardware_interface/PositionJointInterface</hardwareInterface>
-        </joint>
-        <actuator name="motor_2">
-            <hardwareInterface>hardware_interface/PositionJointInterface</hardwareInterface>
-            <mechanicalReduction>1</mechanicalReduction>
-        </actuator>
-    </transmission>
-    <transmission name="transmission_3">
-        <type>transmission_interface/SimpleTransmission</type>
-        <joint name="joint_3">
-            <hardwareInterface>hardware_interface/PositionJointInterface</hardwareInterface>
-        </joint>
-        <actuator name="motor_3">
-            <hardwareInterface>hardware_interface/PositionJointInterface</hardwareInterface>
-            <mechanicalReduction>1</mechanicalReduction>
-        </actuator>
-    </transmission>
-    <transmission name="transmission_4">
-        <type>transmission_interface/SimpleTransmission</type>
-        <joint name="joint_4">
-            <hardwareInterface>hardware_interface/PositionJointInterface</hardwareInterface>
-        </joint>
-        <actuator name="motor_4">
-            <hardwareInterface>hardware_interface/PositionJointInterface</hardwareInterface>
-            <mechanicalReduction>1</mechanicalReduction>
-        </actuator>
-    </transmission>
-    <transmission name="transmission_5">
-        <type>transmission_interface/SimpleTransmission</type>
-        <joint name="joint_5">
-            <hardwareInterface>hardware_interface/PositionJointInterface</hardwareInterface>
-        </joint>
-        <actuator name="motor_5">
-            <hardwareInterface>hardware_interface/PositionJointInterface</hardwareInterface>
-            <mechanicalReduction>1</mechanicalReduction>
-        </actuator>
-    </transmission>
-    <!-- ros_control plugin -->
+    <xacro:default_transmission number="1"/>
+    <xacro:default_transmission number="2"/>
+    <xacro:default_transmission number="3"/>
+    <xacro:default_transmission number="4"/>
+    <xacro:default_transmission number="5"/>
+    <!-- gazebo ros_control plugin -->
     <gazebo>
         <plugin name="gazebo_ros_control" filename="libgazebo_ros_control.so">

Commit message: license update and error fixing oon startup

File: arduinobot_ws/src/arduinobot_description/urdf/arduinobot.urdf (robot description, URDF)
Before this commit: robot arduinobot, 9 links, 8 joints
Links:
- link base_plate: geometry collision mesh filename=package://arduinobot_description/mesh/base_plate.STL scale=0.01 0.01 0.01; visual mesh filename=package://arduinobot_description/mesh/base_plate.STL scale=0.01 0.01 0.01
Joints:
- joint joint_1: limit lower=-1.5707963268 upper=1.5707963268 effort=30 velocity=0.5 -> lower=-1.5707963268 upper=1.5707963268 effort=30 velocity=10
- joint joint_2: limit lower=-1.5707963268 upper=1.5707963268 effort=30 velocity=0.5 -> lower=-1.5707963268 upper=1.5707963268 effort=30 velocity=10
- joint joint_3: limit lower=-1.5707963268 upper=1.5707963268 effort=30 velocity=0.5 -> lower=-1.5707963268 upper=1.5707963268 effort=30 velocity=10
- joint joint_4: limit lower=-1.5707963268 upper=0 effort=30 velocity=0.5 -> lower=-1.5707963268 upper=0 effort=30 velocity=10
- joint joint_5: limit lower=0 upper=1.5707963268 effort=30 velocity=0.5 -> lower=0 upper=1.5707963268 effort=30 velocity=10
- joint virtual_joint: origin xyz=0 0 0.25 -> xyz=0 0 0 rpy=0 0 0
