Commit message: first hardware interface version

File: arduinobot_ws/src/arduinobot_description/urdf/arduinobot_gazebo.xacro (robot description, xacro)
@@ -11,6 +11,6 @@
       </plugin>
     </gazebo>
-    <!-- ros2_control Joint Interface I/O-->
-    <ros2_control name="GazeboSystem" type="system">
+    <!-- ros2_control Gazebo Joint Interface I/O-->
+    <!-- <ros2_control name="GazeboSystem" type="system">
       <hardware>
         <plugin>gazebo_ros2_control/GazeboSystem</plugin>
@@ -52,4 +52,47 @@
         </command_interface>
       </joint>
+    </ros2_control> -->
+    <!-- ros2_control Real Robot Joint Interface I/O-->
+    <ros2_control name="RealRobot" type="system">
+      <hardware>
+        <plugin>arduinobot_controller/ArduinobotInterface</plugin>
+        <param name="port">/dev/ttyUSB0</param>
+      </hardware>
+      <joint name="joint_1">
+        <command_interface name="position">
+          <param name="min">${joint_arm_lower_limit}</param>
+          <param name="max">${joint_arm_upper_limit}</param>
+        </command_interface>
+        <state_interface name="position"/>
+      </joint>
+      <joint name="joint_2">
+        <command_interface name="position">
+          <param name="min">${joint_arm_lower_limit}</param>
+          <param name="max">${joint_arm_upper_limit}</param>
+        </command_interface>
+        <state_interface name="position"/>
+      </joint>
+      <joint name="joint_3">
+        <command_interface name="position">
+          <param name="min">${joint_arm_lower_limit}</param>
+          <param name="max">${joint_arm_upper_limit}</param>
+        </command_interface>
+        <state_interface name="position"/>
+      </joint>
+      <joint name="joint_4">
+        <command_interface name="position">
+          <param name="min">${joint_finger_right_lower_limit}</param>
+          <param name="max">${joint_finger_right_upper_limit}</param>
+        </command_interface>
+        <state_interface name="position"/>
+      </joint>
+      <joint name="joint_5">
+        <param name="mimic">joint_4</param>
+        <param name="multiplier">-1</param>
+        <command_interface name="position">
+          <param name="min">${joint_finger_left_lower_limit}</param>
+          <param name="max">${joint_finger_left_upper_limit}</param>
+        </command_interface>
+      </joint>
     </ros2_control>
 </robot>
