Commit message: model spawned in gazebo

File: arduinobot_ws/src/arduinobot_description/urdf/arduinobot.urdf.xacro (robot description, xacro)
@@ -3,12 +3,26 @@
     <!-- Useful Variables (Properties) -->
     <xacro:property name="PI" value="3.14159265359" />
-    <xacro:property name="low_limit_base_plate_rotation" value="-${PI/2}" />
-    <xacro:property name="up_limit_base_plate_rotation" value="${PI/2}" />
-    <xacro:property name="low_limit_forward_drive_arm_rotation" value="-${PI/2}" />
-    <xacro:property name="up_limit_forward_drive_arm_rotation" value="${PI/2}" />
-    <xacro:property name="low_limit_horizontal_arm_rotation" value="-${PI/2}" />
-    <xacro:property name="up_limit_horizontal_arm_arm_rotation" value="${PI/2}" />
     <!-- Links -->
+    <!-- Used for fixing robot to Gazebo 'base_link' -->
+    <link name="world"/>
+    <joint name="fixed" type="fixed">
+        <parent link="world"/>
+        <child link="base_link"/>
+    </joint>
     <link name="base_link">
+        <inertial>
+            <origin
+                xyz="-0.00377490175092598 0.0117968193300164 0.111915553022725"
+                rpy="0 0 0" />
+            <mass
+                value="0.0497217748522043" />
+            <inertia
+                ixx="2.7691005915736E-05"
+                ixy="3.52926313057377E-10"
+                ixz="2.67965631475746E-09"
+                iyy="4.56375668926374E-05"
+                iyz="1.08925829164701E-07"
+                izz="2.5397344287959E-05" />
+        </inertial>
         <visual>
             <origin rpy="0 0 0" xyz="-0.5 -0.5 0"/>
@@ -25,4 +39,18 @@
     </link>
     <link name="base_plate">
+        <inertial>
+            <origin
+                xyz="-0.00377490175092598 0.0117968193300164 0.111915553022725"
+                rpy="0 0 0" />
+            <mass
+                value="0.0497217748522043" />
+            <inertia
+                ixx="2.7691005915736E-05"
+                ixy="3.52926313057377E-10"
+                ixz="2.67965631475746E-09"
+                iyy="4.56375668926374E-05"
+                iyz="1.08925829164701E-07"
+                izz="2.5397344287959E-05" />
+        </inertial>
         <visual>
             <origin rpy="0 0 0" xyz="-0.39 -0.39 -0.56"/>
@@ -39,4 +67,18 @@
     </link>
     <link name="forward_drive_arm">
+        <inertial>
+            <origin
+                xyz="-0.00377490175092598 0.0117968193300164 0.111915553022725"
+                rpy="0 0 0" />
+            <mass
+                value="0.0497217748522043" />
+            <inertia
+                ixx="2.7691005915736E-05"
+                ixy="3.52926313057377E-10"
+                ixz="2.67965631475746E-09"
+                iyy="4.56375668926374E-05"
+                iyz="1.08925829164701E-07"
+                izz="2.5397344287959E-05" />
+        </inertial>
         <visual>
             <origin rpy=" 0 -${PI/2} ${PI/2}" xyz="0.19 0.06 -0.08"/>
@@ -53,4 +95,18 @@
     </link>
     <link name="horizontal_arm">
+        <inertial>
+            <origin
+                xyz="-0.00377490175092598 0.0117968193300164 0.111915553022725"
+                rpy="0 0 0" />
+            <mass
+                value="0.0497217748522043" />
+            <inertia
+                ixx="2.7691005915736E-05"
+                ixy="3.52926313057377E-10"
+                ixz="2.67965631475746E-09"
+                iyy="4.56375668926374E-05"
+                iyz="1.08925829164701E-07"
+                izz="2.5397344287959E-05" />
+        </inertial>
         <visual>
             <origin rpy="${PI/2} 0 ${PI/2}" xyz="-0.03 -0.4 -0.06"/>
@@ -67,4 +123,18 @@
     </link>
     <link name="claw_support">
+        <inertial>
+            <origin
+                xyz="-0.00377490175092598 0.0117968193300164 0.111915553022725"
+                rpy="0 0 0" />
+            <mass
+                value="0.0497217748522043" />
+            <inertia
+                ixx="2.7691005915736E-05"
+                ixy="3.52926313057377E-10"
+                ixz="2.67965631475746E-09"
+                iyy="4.56375668926374E-05"
+                iyz="1.08925829164701E-07"
+                izz="2.5397344287959E-05" />
+        </inertial>
         <visual>
             <origin rpy="0 0 ${PI/2}" xyz="0 -0.05 -0.15"/>
@@ -81,4 +151,18 @@
     </link>
     <link name="gripper_right">
+        <inertial>
+            <origin
+                xyz="-0.00377490175092598 0.0117968193300164 0.111915553022725"
+                rpy="0 0 0" />
+            <mass
+                value="0.0497217748522043" />
+            <inertia
+                ixx="2.7691005915736E-05"
+                ixy="3.52926313057377E-10"
+                ixz="2.67965631475746E-09"
+                iyy="4.56375668926374E-05"
+                iyz="1.08925829164701E-07"
+                izz="2.5397344287959E-05" />
+        </inertial>
         <visual>
             <origin rpy="0 0 -${PI/2}" xyz="-0.1 0.50 -0.1"/>
@@ -95,4 +179,18 @@
     </link>
     <link name="gripper_left">
+        <inertial>
+            <origin
+                xyz="-0.00377490175092598 0.0117968193300164 0.111915553022725"
+                rpy="0 0 0" />
+            <mass
+                value="0.0497217748522043" />
+            <inertia
+                ixx="2.7691005915736E-05"
+                ixy="3.52926313057377E-10"
+                ixz="2.67965631475746E-09"
+                iyy="4.56375668926374E-05"
+                iyz="1.08925829164701E-07"
+                izz="2.5397344287959E-05" />
+        </inertial>
         <visual>
             <origin rpy="0 0 -${PI/2}" xyz="-0.04 0.50 -0.1"/>
@@ -156,3 +254,52 @@
         <origin xyz="0 0 0"/>
     </joint>
+    <!-- Transmissions-->
+    <transmission name="transmission_1">
+        <type>transmission_interface/SimpleTransmission</type>
+        <joint name="joint_1">
+            <hardwareInterface>hardware_interface/EffortJointInterface</hardwareInterface>
+        </joint>
+        <actuator name="motor_1">
+            <hardwareInterface>hardware_interface/EffortJointInterface</hardwareInterface>
+            <mechanicalReduction>1</mechanicalReduction>
+        </actuator>
+    </transmission>
+    <transmission name="transmission_2">
+        <type>transmission_interface/SimpleTransmission</type>
+        <joint name="joint_2">
+            <hardwareInterface>hardware_interface/EffortJointInterface</hardwareInterface>
+        </joint>
+        <actuator name="motor_2">
+            <hardwareInterface>hardware_interface/EffortJointInterface</hardwareInterface>
+            <mechanicalReduction>1</mechanicalReduction>
+        </actuator>
+    </transmission>
+    <transmission name="transmission_3">
+        <type>transmission_interface/SimpleTransmission</type>
+        <joint name="joint_3">
+            <hardwareInterface>hardware_interface/EffortJointInterface</hardwareInterface>
+        </joint>
+        <actuator name="motor_3">
+            <hardwareInterface>hardware_interface/EffortJointInterface</hardwareInterface>
+            <mechanicalReduction>1</mechanicalReduction>
+        </actuator>
+    </transmission>
+    <transmission name="transmission_4">
+        <type>transmission_interface/SimpleTransmission</type>
+        <joint name="joint_4">
+            <hardwareInterface>hardware_interface/EffortJointInterface</hardwareInterface>
+        </joint>
+        <actuator name="motor_4">
+            <hardwareInterface>hardware_interface/EffortJointInterface</hardwareInterface>
+            <mechanicalReduction>1</mechanicalReduction>
+        </actuator>
+    </transmission>
+    <!-- ros_control plugin -->
+    <gazebo>
+        <plugin name="gazebo_ros_control" filename="libgazebo_ros_control.so">
+            <robotNamespace>/arduinobot</robotNamespace>
+            <robotSimType>gazebo_ros_control/DefaultRobotHWSim</robotSimType>
+            <legacyModeNS>true</legacyModeNS>
+        </plugin>
+    </gazebo>
 </robot>

Commit message: first working version of the gazebo sim

File: arduinobot_ws/src/arduinobot_description/urdf/arduinobot.urdf.xacro (robot description, xacro)
@@ -4,24 +4,10 @@
     <xacro:property name="PI" value="3.14159265359" />
     <!-- Links -->
-    <!-- Used for fixing robot to Gazebo 'base_link' -->
-    <link name="world"/>
-    <joint name="fixed" type="fixed">
-        <parent link="world"/>
-        <child link="base_link"/>
-    </joint>
     <link name="base_link">
         <inertial>
-            <origin
-                xyz="-0.00377490175092598 0.0117968193300164 0.111915553022725"
-                rpy="0 0 0" />
-            <mass
-                value="0.0497217748522043" />
-            <inertia
-                ixx="2.7691005915736E-05"
-                ixy="3.52926313057377E-10"
-                ixz="2.67965631475746E-09"
-                iyy="4.56375668926374E-05"
-                iyz="1.08925829164701E-07"
-                izz="2.5397344287959E-05" />
+                <mass value="1" />
+                <inertia ixx="1.0" ixy="0.0" ixz="0.0"
+                     iyy="1.0" iyz="0.0"
+                     izz="1.0" />
         </inertial>
         <visual>
@@ -40,16 +26,8 @@
     <link name="base_plate">
         <inertial>
-            <origin
-                xyz="-0.00377490175092598 0.0117968193300164 0.111915553022725"
-                rpy="0 0 0" />
-            <mass
-                value="0.0497217748522043" />
-            <inertia
-                ixx="2.7691005915736E-05"
-                ixy="3.52926313057377E-10"
-                ixz="2.67965631475746E-09"
-                iyy="4.56375668926374E-05"
-                iyz="1.08925829164701E-07"
-                izz="2.5397344287959E-05" />
+                <mass value="1" />
+                <inertia ixx="1.0" ixy="0.0" ixz="0.0"
+                     iyy="1.0" iyz="0.0"
+                     izz="1.0" />
         </inertial>
         <visual>
@@ -68,16 +46,8 @@
     <link name="forward_drive_arm">
         <inertial>
-            <origin
-                xyz="-0.00377490175092598 0.0117968193300164 0.111915553022725"
-                rpy="0 0 0" />
-            <mass
-                value="0.0497217748522043" />
-            <inertia
-                ixx="2.7691005915736E-05"
-                ixy="3.52926313057377E-10"
-                ixz="2.67965631475746E-09"
-                iyy="4.56375668926374E-05"
-                iyz="1.08925829164701E-07"
-                izz="2.5397344287959E-05" />
+                <mass value="1" />
+                <inertia ixx="1.0" ixy="0.0" ixz="0.0"
+                     iyy="1.0" iyz="0.0"
+                     izz="1.0" />
         </inertial>
         <visual>
@@ -96,16 +66,8 @@
     <link name="horizontal_arm">
         <inertial>
-            <origin
-                xyz="-0.00377490175092598 0.0117968193300164 0.111915553022725"
-                rpy="0 0 0" />
-            <mass
-                value="0.0497217748522043" />
-            <inertia
-                ixx="2.7691005915736E-05"
-                ixy="3.52926313057377E-10"
-                ixz="2.67965631475746E-09"
-                iyy="4.56375668926374E-05"
-                iyz="1.08925829164701E-07"
-                izz="2.5397344287959E-05" />
+                <mass value="1" />
+                <inertia ixx="1.0" ixy="0.0" ixz="0.0"
+                     iyy="1.0" iyz="0.0"
+                     izz="1.0" />
         </inertial>
         <visual>
@@ -124,16 +86,8 @@
     <link name="claw_support">
         <inertial>
-            <origin
-                xyz="-0.00377490175092598 0.0117968193300164 0.111915553022725"
-                rpy="0 0 0" />
-            <mass
-                value="0.0497217748522043" />
-            <inertia
-                ixx="2.7691005915736E-05"
-                ixy="3.52926313057377E-10"
-                ixz="2.67965631475746E-09"
-                iyy="4.56375668926374E-05"
-                iyz="1.08925829164701E-07"
-                izz="2.5397344287959E-05" />
+                <mass value="1" />
+                <inertia ixx="1.0" ixy="0.0" ixz="0.0"
+                     iyy="1.0" iyz="0.0"
+                     izz="1.0" />
         </inertial>
         <visual>
@@ -152,16 +106,8 @@
     <link name="gripper_right">
         <inertial>
-            <origin
-                xyz="-0.00377490175092598 0.0117968193300164 0.111915553022725"
-                rpy="0 0 0" />
-            <mass
-                value="0.0497217748522043" />
-            <inertia
-                ixx="2.7691005915736E-05"
-                ixy="3.52926313057377E-10"
-                ixz="2.67965631475746E-09"
-                iyy="4.56375668926374E-05"
-                iyz="1.08925829164701E-07"
-                izz="2.5397344287959E-05" />
+                <mass value="1" />
+                <inertia ixx="1.0" ixy="0.0" ixz="0.0"
+                     iyy="1.0" iyz="0.0"
+                     izz="1.0" />
         </inertial>
         <visual>
@@ -180,16 +126,8 @@
     <link name="gripper_left">
         <inertial>
-            <origin
-                xyz="-0.00377490175092598 0.0117968193300164 0.111915553022725"
-                rpy="0 0 0" />
-            <mass
-                value="0.0497217748522043" />
-            <inertia
-                ixx="2.7691005915736E-05"
-                ixy="3.52926313057377E-10"
-                ixz="2.67965631475746E-09"
-                iyy="4.56375668926374E-05"
-                iyz="1.08925829164701E-07"
-                izz="2.5397344287959E-05" />
+                <mass value="1" />
+                <inertia ixx="1.0" ixy="0.0" ixz="0.0"
+                     iyy="1.0" iyz="0.0"
+                     izz="1.0" />
         </inertial>
         <visual>
@@ -200,5 +138,5 @@
         </visual>
         <collision>
-            <origin rpy="0 0 -${PI/2}" xyz="-0.2 0.50 -0.1"/>
+            <origin rpy="0 0 -${PI/2}" xyz="-0.04 0.50 -0.1"/>
             <geometry>
                 <mesh filename="package://arduinobot_description/mesh/left_finger.STL" scale="0.01 0.01 0.01"/>
@@ -258,8 +196,7 @@
         <type>transmission_interface/SimpleTransmission</type>
         <joint name="joint_1">
-            <hardwareInterface>hardware_interface/EffortJointInterface</hardwareInterface>
+            <hardwareInterface>hardware_interface/PositionJointInterface</hardwareInterface>
         </joint>
         <actuator name="motor_1">
-            <hardwareInterface>hardware_interface/EffortJointInterface</hardwareInterface>
             <mechanicalReduction>1</mechanicalReduction>
         </actuator>
@@ -268,8 +205,7 @@
         <type>transmission_interface/SimpleTransmission</type>
         <joint name="joint_2">
-            <hardwareInterface>hardware_interface/EffortJointInterface</hardwareInterface>
+            <hardwareInterface>hardware_interface/PositionJointInterface</hardwareInterface>
         </joint>
         <actuator name="motor_2">
-            <hardwareInterface>hardware_interface/EffortJointInterface</hardwareInterface>
             <mechanicalReduction>1</mechanicalReduction>
         </actuator>
@@ -278,8 +214,7 @@
         <type>transmission_interface/SimpleTransmission</type>
         <joint name="joint_3">
-            <hardwareInterface>hardware_interface/EffortJointInterface</hardwareInterface>
+            <hardwareInterface>hardware_interface/PositionJointInterface</hardwareInterface>
         </joint>
         <actuator name="motor_3">
-            <hardwareInterface>hardware_interface/EffortJointInterface</hardwareInterface>
             <mechanicalReduction>1</mechanicalReduction>
         </actuator>
@@ -288,8 +223,7 @@
         <type>transmission_interface/SimpleTransmission</type>
         <joint name="joint_4">
-            <hardwareInterface>hardware_interface/EffortJointInterface</hardwareInterface>
+            <hardwareInterface>hardware_interface/PositionJointInterface</hardwareInterface>
         </joint>
         <actuator name="motor_4">
-            <hardwareInterface>hardware_interface/EffortJointInterface</hardwareInterface>
             <mechanicalReduction>1</mechanicalReduction>
         </actuator>

Commit message: creation and spawn of gazebo sim controllers

File: arduinobot_ws/src/arduinobot_description/urdf/arduinobot.urdf.xacro (robot description, xacro)
@@ -4,4 +4,10 @@
     <xacro:property name="PI" value="3.14159265359" />
     <!-- Links -->
+    <link name="world"/>
+    <joint name="fixed" type="fixed">
+        <parent link="world"/>
+        <child link="base_link"/>
+        <origin xyz="0 0 0.25"/>
+    </joint>
     <link name="base_link">
         <inertial>
@@ -26,5 +32,5 @@
     <link name="base_plate">
         <inertial>
-                <mass value="1" />
+                <mass value="0.1" />
                 <inertia ixx="1.0" ixy="0.0" ixz="0.0"
                      iyy="1.0" iyz="0.0"
@@ -46,5 +52,5 @@
     <link name="forward_drive_arm">
         <inertial>
-                <mass value="1" />
+                <mass value="0.1" />
                 <inertia ixx="1.0" ixy="0.0" ixz="0.0"
                      iyy="1.0" iyz="0.0"
@@ -66,5 +72,5 @@
     <link name="horizontal_arm">
         <inertial>
-                <mass value="1" />
+                <mass value="0.1" />
                 <inertia ixx="1.0" ixy="0.0" ixz="0.0"
                      iyy="1.0" iyz="0.0"
@@ -86,5 +92,5 @@
     <link name="claw_support">
         <inertial>
-                <mass value="1" />
+                <mass value="0.1" />
                 <inertia ixx="1.0" ixy="0.0" ixz="0.0"
                      iyy="1.0" iyz="0.0"
@@ -106,5 +112,5 @@
     <link name="gripper_right">
         <inertial>
-                <mass value="1" />
+                <mass value="0.1" />
                 <inertia ixx="1.0" ixy="0.0" ixz="0.0"
                      iyy="1.0" iyz="0.0"
@@ -126,5 +132,5 @@
     <link name="gripper_left">
         <inertial>
-                <mass value="1" />
+                <mass value="0.1" />
                 <inertia ixx="1.0" ixy="0.0" ixz="0.0"
                      iyy="1.0" iyz="0.0"
@@ -151,5 +157,5 @@
         <origin xyz="0 0 0.307"/>
         <axis xyz="0 0 1"/>
-        <limit lower="-${PI/2}" upper="${PI/2}" effort="1000.0" velocity="0.5"/>
+        <limit lower="-${PI/2}" upper="${PI/2}" effort="30.0" velocity="0.5"/>
     </joint>
     <joint name ="joint_2" type="revolute">
@@ -158,5 +164,5 @@
         <origin xyz="0 0 0.28"/>
         <axis xyz="1 0 0"/>
-        <limit lower="-${PI/2}" upper="${PI/2}" effort="1000.0" velocity="0.5"/>
+        <limit lower="-${PI/2}" upper="${PI/2}" effort="30.0" velocity="0.5"/>
     </joint>
     <joint name ="joint_3" type="revolute">
@@ -165,5 +171,5 @@
         <origin xyz="0 0 0.8"/>
         <axis xyz="1 0 0"/>
-        <limit lower="-${PI/2}" upper="${PI/2}" effort="1000.0" velocity="0.5"/>
+        <limit lower="-${PI/2}" upper="${PI/2}" effort="30.0" velocity="0.5"/>
     </joint>
     <joint name ="horizontal_arm_to_claw_support" type="fixed">
@@ -177,5 +183,5 @@
         <origin xyz="-0.04 0.13 -0.1"/>
         <axis xyz="0 0 1"/>
-        <limit lower="-${PI/2}" upper="0" effort="1000.0" velocity="0.5"/>
+        <limit lower="-${PI/2}" upper="0" effort="30.0" velocity="0.5"/>
     </joint>
     <joint name ="joint_5" type="revolute">
@@ -184,5 +190,5 @@
         <origin xyz="-0.22 0.13 -0.1"/>
         <axis xyz="0 0 1"/>
-        <limit lower="0" upper="${PI/2}" effort="1000.0" velocity="0.5"/>
+        <limit lower="0" upper="${PI/2}" effort="30.0" velocity="0.5"/>
         <mimic joint="joint_4" multiplier="-1" offset="0"/>
     </joint>
@@ -196,7 +202,8 @@
         <type>transmission_interface/SimpleTransmission</type>
         <joint name="joint_1">
-            <hardwareInterface>hardware_interface/PositionJointInterface</hardwareInterface>
+            <hardwareInterface>hardware_interface/EffortJointInterface</hardwareInterface>
         </joint>
         <actuator name="motor_1">
+            <hardwareInterface>hardware_interface/EffortJointInterface</hardwareInterface>
             <mechanicalReduction>1</mechanicalReduction>
         </actuator>
@@ -205,7 +212,8 @@
         <type>transmission_interface/SimpleTransmission</type>
         <joint name="joint_2">
-            <hardwareInterface>hardware_interface/PositionJointInterface</hardwareInterface>
+            <hardwareInterface>hardware_interface/EffortJointInterface</hardwareInterface>
         </joint>
         <actuator name="motor_2">
+            <hardwareInterface>hardware_interface/EffortJointInterface</hardwareInterface>
             <mechanicalReduction>1</mechanicalReduction>
         </actuator>
@@ -214,7 +222,8 @@
         <type>transmission_interface/SimpleTransmission</type>
         <joint name="joint_3">
-            <hardwareInterface>hardware_interface/PositionJointInterface</hardwareInterface>
+            <hardwareInterface>hardware_interface/EffortJointInterface</hardwareInterface>
         </joint>
         <actuator name="motor_3">
+            <hardwareInterface>hardware_interface/EffortJointInterface</hardwareInterface>
             <mechanicalReduction>1</mechanicalReduction>
         </actuator>
@@ -223,7 +232,8 @@
         <type>transmission_interface/SimpleTransmission</type>
         <joint name="joint_4">
-            <hardwareInterface>hardware_interface/PositionJointInterface</hardwareInterface>
+            <hardwareInterface>hardware_interface/EffortJointInterface</hardwareInterface>
         </joint>
         <actuator name="motor_4">
+            <hardwareInterface>hardware_interface/EffortJointInterface</hardwareInterface>
             <mechanicalReduction>1</mechanicalReduction>
         </actuator>

Commit message: created fake control interface with the gazebo controller and integration with mveit

File: arduinobot_ws/src/arduinobot_description/urdf/arduinobot.urdf.xacro (robot description, xacro)
@@ -5,5 +5,5 @@
     <!-- Links -->
     <link name="world"/>
-    <joint name="fixed" type="fixed">
+    <joint name="virtual_joint" type="fixed">
         <parent link="world"/>
         <child link="base_link"/>
@@ -239,8 +239,18 @@
         </actuator>
     </transmission>
+    <transmission name="transmission_5">
+        <type>transmission_interface/SimpleTransmission</type>
+        <joint name="joint_5">
+            <hardwareInterface>hardware_interface/EffortJointInterface</hardwareInterface>
+        </joint>
+        <actuator name="motor_5">
+            <hardwareInterface>hardware_interface/EffortJointInterface</hardwareInterface>
+            <mechanicalReduction>1</mechanicalReduction>
+        </actuator>
+    </transmission>
     <!-- ros_control plugin -->
     <gazebo>
         <plugin name="gazebo_ros_control" filename="libgazebo_ros_control.so">
-            <robotNamespace>/arduinobot</robotNamespace>
+            <robotNamespace>/arduinobot_sim</robotNamespace>
             <robotSimType>gazebo_ros_control/DefaultRobotHWSim</robotSimType>
             <legacyModeNS>true</legacyModeNS>
