Commit message: moveit migration

File: arduinobot_ws/src/arduinobot_description/urdf/arduinobot.urdf.xacro (robot description, xacro)
@@ -1,8 +1,6 @@
 <?xml version="1.0"?>
 <robot xmlns:xacro="http://www.ros.org/wiki/xacro" name="arduinobot">
-    <!-- Useful Variables (Properties) -->
-    <xacro:property name="PI" value="3.14159265359" />
-    <xacro:property name="effort" value="30" />
-    <xacro:property name="velocity" value="10" />
+    <!-- Include XACRO Variables -->
+    <xacro:include filename="$(find arduinobot_description)/urdf/arduinobot_variables.xacro" />
     <!-- Include Gazebo Parameters -->
     <xacro:include filename="$(find arduinobot_description)/urdf/arduinobot_gazebo.xacro" />
@@ -145,5 +143,6 @@
         <origin xyz="0 0 0.307"/>
         <axis xyz="0 0 1"/>
-        <limit lower="-${PI / 2}" upper="${PI / 2}" effort="${effort}" velocity="${velocity}"/>
+        <limit lower="${joint_arm_lower_limit}" upper="${joint_arm_upper_limit}"
+               effort="${effort}" velocity="${velocity}"/>
     </joint>
     <joint name ="joint_2" type="revolute">
@@ -152,5 +151,6 @@
         <origin xyz="-0.02 0 0.35"/>
         <axis xyz="1 0 0"/>
-        <limit lower="-${PI / 2}" upper="${PI / 2}" effort="${effort}" velocity="${velocity}"/>
+        <limit lower="${joint_arm_lower_limit}" upper="${joint_arm_upper_limit}"
+                effort="${effort}" velocity="${velocity}"/>
     </joint>
     <joint name ="joint_3" type="revolute">
@@ -159,5 +159,6 @@
         <origin xyz="0 0 0.8"/>
         <axis xyz="1 0 0"/>
-        <limit lower="-${PI / 2}" upper="${PI / 2}" effort="${effort}" velocity="${velocity}"/>
+        <limit lower="${joint_arm_lower_limit}" upper="${joint_arm_upper_limit}"
+               effort="${effort}" velocity="${velocity}"/>
     </joint>
     <joint name ="horizontal_arm_to_claw_support" type="fixed">
@@ -171,5 +172,6 @@
         <origin xyz="-0.04 0.13 -0.1"/>
         <axis xyz="0 0 1"/>
-        <limit lower="-${PI / 2}" upper="0" effort="${effort}" velocity="${velocity}"/>
+        <limit lower="${joint_finger_right_lower_limit}" upper="${joint_finger_right_upper_limit}"
+               effort="${effort}" velocity="${velocity}"/>
     </joint>
     <joint name ="joint_5" type="revolute">
@@ -178,5 +180,6 @@
         <origin xyz="-0.22 0.13 -0.1"/>
         <axis xyz="0 0 1"/>
-        <limit lower="0" upper="${PI / 2}" effort="${effort}" velocity="${velocity}"/>
+        <limit lower="${joint_finger_left_lower_limit}" upper="${joint_finger_left_upper_limit}"
+               effort="${effort}" velocity="${velocity}"/>
     </joint>
     <joint name ="gripper_right_to_tool" type="fixed">

File: arduinobot_ws/src/arduinobot_description/urdf/arduinobot_gazebo.xacro (robot description, xacro)
@@ -1,5 +1,7 @@
 <?xml version="1.0"?>
 <robot xmlns:xacro="http://www.ros.org/wiki/xacro" name="arduinobot">
-    <!-- gazebo ros2_control plugin -->
+    <!-- Include XACRO Variables -->
+    <xacro:include filename="$(find arduinobot_description)/urdf/arduinobot_variables.xacro" />
+    <!-- Gazebo ros2_control plugin -->
     <gazebo>
       <plugin filename="libgazebo_ros2_control.so" name="gazebo_ros2_control">
@@ -9,4 +11,5 @@
       </plugin>
     </gazebo>
+    <!-- ros2_control Joint Interface I/O-->
     <ros2_control name="GazeboSystem" type="system">
       <hardware>
@@ -15,6 +18,6 @@
       <joint name="joint_1">
         <command_interface name="position">
-          <param name="min">-1</param>
-          <param name="max">1</param>
+          <param name="min">${joint_arm_lower_limit}</param>
+          <param name="max">${joint_arm_upper_limit}</param>
         </command_interface>
         <state_interface name="position"/>
@@ -22,6 +25,6 @@
       <joint name="joint_2">
         <command_interface name="position">
-          <param name="min">-1</param>
-          <param name="max">1</param>
+          <param name="min">${joint_arm_lower_limit}</param>
+          <param name="max">${joint_arm_upper_limit}</param>
         </command_interface>
         <state_interface name="position"/>
@@ -29,6 +32,6 @@
       <joint name="joint_3">
         <command_interface name="position">
-          <param name="min">-1</param>
-          <param name="max">1</param>
+          <param name="min">${joint_arm_lower_limit}</param>
+          <param name="max">${joint_arm_upper_limit}</param>
         </command_interface>
         <state_interface name="position"/>
@@ -36,6 +39,6 @@
       <joint name="joint_4">
         <command_interface name="position">
-          <param name="min">-1</param>
-          <param name="max">1</param>
+          <param name="min">${joint_finger_right_lower_limit}</param>
+          <param name="max">${joint_finger_right_upper_limit}</param>
         </command_interface>
         <state_interface name="position"/>
@@ -45,6 +48,6 @@
         <param name="multiplier">-1</param>
         <command_interface name="position">
-          <param name="min">-1</param>
-          <param name="max">1</param>
+          <param name="min">${joint_finger_left_lower_limit}</param>
+          <param name="max">${joint_finger_left_upper_limit}</param>
         </command_interface>
         <state_interface name="position"/>

Commit message: moveit planning

File: arduinobot_ws/src/arduinobot_description/urdf/arduinobot.urdf.xacro (robot description, xacro)
@@ -182,4 +182,5 @@
         <limit lower="${joint_finger_left_lower_limit}" upper="${joint_finger_left_upper_limit}"
                effort="${effort}" velocity="${velocity}"/>
+        <mimic joint="joint_4" multiplier="-1"/>
     </joint>
     <joint name ="gripper_right_to_tool" type="fixed">

File: arduinobot_ws/src/arduinobot_description/urdf/arduinobot_gazebo.xacro (robot description, xacro)
@@ -51,5 +51,4 @@
           <param name="max">${joint_finger_left_upper_limit}</param>
         </command_interface>
-        <state_interface name="position"/>
       </joint>
     </ros2_control>

File: arduinobot_ws/src/arduinobot_moveit/config/arduinobot.urdf.xacro (robot description, xacro)
@@ -1,9 +1,5 @@
 <?xml version="1.0"?>
 <robot xmlns:xacro="http://www.ros.org/wiki/xacro" name="arduinobot">
-    <xacro:arg name="initial_positions_file" default="initial_positions.yaml" />
     <!-- Import arduinobot urdf file -->
     <xacro:include filename="$(find arduinobot_description)/urdf/arduinobot.urdf.xacro" />
-    <!-- Import control_xacro -->
-    <xacro:include filename="arduinobot.ros2_control.xacro" />
-    <xacro:arduinobot_ros2_control name="FakeSystem" initial_positions_file="$(arg initial_positions_file)"/>
 </robot>

Commit message: added bringup

File: arduinobot_ws/src/arduinobot_description/urdf/arduinobot.urdf.xacro (robot description, xacro)
@@ -1,8 +1,12 @@
 <?xml version="1.0"?>
 <robot xmlns:xacro="http://www.ros.org/wiki/xacro" name="arduinobot">
+    <!-- Load Simulated or Real Hardware Interfaces -->
+    <xacro:arg name="is_sim" default="true"/>
     <!-- Include XACRO Variables -->
     <xacro:include filename="$(find arduinobot_description)/urdf/arduinobot_variables.xacro" />
     <!-- Include Gazebo Parameters -->
     <xacro:include filename="$(find arduinobot_description)/urdf/arduinobot_gazebo.xacro" />
+    <!-- Include ros2_control Plugins -->
+    <xacro:include filename="$(find arduinobot_description)/urdf/arduinobot_ros2_control.xacro" />
     <!-- Useful Macros -->
     <xacro:macro name="default_inertial" params="mass">

File: arduinobot_ws/src/arduinobot_description/urdf/arduinobot_gazebo.xacro (robot description, xacro)
@@ -11,88 +11,3 @@
       </plugin>
     </gazebo>
-    <!-- ros2_control Gazebo Joint Interface I/O-->
-    <!-- <ros2_control name="GazeboSystem" type="system">
-      <hardware>
-        <plugin>gazebo_ros2_control/GazeboSystem</plugin>
-      </hardware>
-      <joint name="joint_1">
-        <command_interface name="position">
-          <param name="min">${joint_arm_lower_limit}</param>
-          <param name="max">${joint_arm_upper_limit}</param>
-        </command_interface>
-        <state_interface name="position"/>
-      </joint>
-      <joint name="joint_2">
-        <command_interface name="position">
-          <param name="min">${joint_arm_lower_limit}</param>
-          <param name="max">${joint_arm_upper_limit}</param>
-        </command_interface>
-        <state_interface name="position"/>
-      </joint>
-      <joint name="joint_3">
-        <command_interface name="position">
-          <param name="min">${joint_arm_lower_limit}</param>
-          <param name="max">${joint_arm_upper_limit}</param>
-        </command_interface>
-        <state_interface name="position"/>
-      </joint>
-      <joint name="joint_4">
-        <command_interface name="position">
-          <param name="min">${joint_finger_right_lower_limit}</param>
-          <param name="max">${joint_finger_right_upper_limit}</param>
-        </command_interface>
-        <state_interface name="position"/>
-      </joint>
-      <joint name="joint_5">
-        <param name="mimic">joint_4</param>
-        <param name="multiplier">-1</param>
-        <command_interface name="position">
-          <param name="min">${joint_finger_left_lower_limit}</param>
-          <param name="max">${joint_finger_left_upper_limit}</param>
-        </command_interface>
-      </joint>
-    </ros2_control> -->
-    <!-- ros2_control Real Robot Joint Interface I/O-->
-    <ros2_control name="RealRobot" type="system">
-      <hardware>
-        <plugin>arduinobot_controller/ArduinobotInterface</plugin>
-        <param name="port">/dev/ttyUSB0</param>
-      </hardware>
-      <joint name="joint_1">
-        <command_interface name="position">
-          <param name="min">${joint_arm_lower_limit}</param>
-          <param name="max">${joint_arm_upper_limit}</param>
-        </command_interface>
-        <state_interface name="position"/>
-      </joint>
-      <joint name="joint_2">
-        <command_interface name="position">
-          <param name="min">${joint_arm_lower_limit}</param>
-          <param name="max">${joint_arm_upper_limit}</param>
-        </command_interface>
-        <state_interface name="position"/>
-      </joint>
-      <joint name="joint_3">
-        <command_interface name="position">
-          <param name="min">${joint_arm_lower_limit}</param>
-          <param name="max">${joint_arm_upper_limit}</param>
-        </command_interface>
-        <state_interface name="position"/>
-      </joint>
-      <joint name="joint_4">
-        <command_interface name="position">
-          <param name="min">${joint_finger_right_lower_limit}</param>
-          <param name="max">${joint_finger_right_upper_limit}</param>
-        </command_interface>
-        <state_interface name="position"/>
-      </joint>
-      <joint name="joint_5">
-        <param name="mimic">joint_4</param>
-        <param name="multiplier">-1</param>
-        <command_interface name="position">
-          <param name="min">${joint_finger_left_lower_limit}</param>
-          <param name="max">${joint_finger_left_upper_limit}</param>
-        </command_interface>
-      </joint>
-    </ros2_control>
 </robot>

Commit message: added missing deps and fix collision origin

File: arduinobot_ws/src/arduinobot_description/urdf/arduinobot.urdf.xacro (robot description, xacro)
@@ -69,5 +69,5 @@
         </visual>
         <collision>
-            <origin rpy=" 0 -${PI / 2} -${PI / 2}" xyz="0.19 0.06 -0.08"/>
+            <origin rpy=" 0 -${PI / 2} ${PI / 2}" xyz="0.19 0.06 -0.08"/>
             <geometry>
                 <mesh filename="package://arduinobot_description/meshes/forward_drive_arm.STL" scale="0.01 0.01 0.01"/>

Commit message: Update arduinobot.urdf.xacro

File: arduinobot_ws/src/arduinobot_description/urdf/arduinobot.urdf.xacro (robot description, xacro)
@@ -1,39 +1,9 @@
-<?xml version="1.0"?>
-<robot xmlns:xacro="http://www.ros.org/wiki/xacro" name="arduinobot">
-    <!-- Load Simulated or Real Hardware Interfaces -->
-    <xacro:arg name="is_sim" default="true"/>
-    <!-- Include XACRO Variables -->
-    <xacro:include filename="$(find arduinobot_description)/urdf/arduinobot_variables.xacro" />
-    <!-- Include Gazebo Parameters -->
-    <xacro:include filename="$(find arduinobot_description)/urdf/arduinobot_gazebo.xacro" />
-    <!-- Include ros2_control Plugins -->
-    <xacro:include filename="$(find arduinobot_description)/urdf/arduinobot_ros2_control.xacro" />
-    <!-- Useful Macros -->
-    <xacro:macro name="default_inertial" params="mass">
-        <inertial>
-            <origin xyz="0 0 0" rpy="0 0 0"/>
-            <mass value="${mass}" />
-            <inertia ixx="1.0" ixy="0.0" ixz="0.0"
-                     iyy="1.0" iyz="0.0"
-                     izz="1.0" />
-        </inertial>
-    </xacro:macro>
-    <xacro:macro name="default_transmission" params="number">
-        <transmission name="transmission_${number}">
-            <plugin>transmission_interface/SimpleTransmission</plugin>
-            <actuator name="motor_${number}" role="actuator1"/>
-            <joint name="wheel_${number}"    role="joint1">
-                <mechanical_reduction>1.0</mechanical_reduction>
-            </joint>
-        </transmission>
-    </xacro:macro>
-    <!-- Links -->
+<robot name="arduinobot">
     <link name="world"/>
     <link name="base_link">
-        <xacro:default_inertial mass="1.0"/>
         <visual>
             <origin rpy="0 0 0" xyz="-0.5 -0.5 0"/>
             <geometry>
-                <mesh filename="package://arduinobot_description/meshes/basement.STL" scale="0.01 0.01 0.01"/>
+                <mesh filename="basement.STL"/>
             </geometry>
         </visual>
@@ -41,100 +11,8 @@
             <origin rpy="0 0 0" xyz="-0.5 -0.5 0"/>
             <geometry>
-                <mesh filename="package://arduinobot_description/meshes/basement.STL" scale="0.01 0.01 0.01"/>
+                <mesh filename="basement.STL"/>
             </geometry>
         </collision>
     </link>
-    <link name="base_plate">
-        <xacro:default_inertial mass="0.1"/>
-        <visual>
-            <origin rpy="0 0 0" xyz="-0.39 -0.39 -0.56"/>
-            <geometry>
-                <mesh filename="package://arduinobot_description/meshes/base_plate.STL" scale="0.01 0.01 0.01"/>
-            </geometry>
-        </visual>
-        <collision>
-            <origin rpy="0 0 0" xyz="-0.39 -0.39 -0.56"/>
-            <geometry>
-                <mesh filename="package://arduinobot_description/meshes/base_plate.STL" scale="0.01 0.01 0.01"/>
-            </geometry>
-        </collision>
-    </link>
-    <link name="forward_drive_arm">
-        <xacro:default_inertial mass="0.1"/>
-        <visual>
-            <origin rpy=" 0 -${PI / 2} ${PI / 2}" xyz="0.19 0.06 -0.08"/>
-            <geometry>
-                <mesh filename="package://arduinobot_description/meshes/forward_drive_arm.STL" scale="0.01 0.01 0.01"/>
-            </geometry>
-        </visual>
-        <collision>
-            <origin rpy=" 0 -${PI / 2} ${PI / 2}" xyz="0.19 0.06 -0.08"/>
-            <geometry>
-                <mesh filename="package://arduinobot_description/meshes/forward_drive_arm.STL" scale="0.01 0.01 0.01"/>
-            </geometry>
-        </collision>
-    </link>
-    <link name="horizontal_arm">
-        <xacro:default_inertial mass="0.1"/>
-        <visual>
-            <origin rpy="${PI / 2} 0 ${PI / 2}" xyz="-0.03 -0.4 -0.06"/>
-            <geometry>
-                <mesh filename="package://arduinobot_description/meshes/horizontal_arm.STL" scale="0.01 0.01 0.01"/>
-            </geometry>
-        </visual>
-        <collision>
-            <origin rpy="${PI / 2} 0 ${PI / 2}" xyz="-0.03 -0.4 -0.06"/>
-            <geometry>
-                <mesh filename="package://arduinobot_description/meshes/horizontal_arm.STL" scale="0.01 0.01 0.01"/>
-            </geometry>
-        </collision>
-    </link>
-    <link name="claw_support">
-        <xacro:default_inertial mass="0.05"/>
-        <visual>
-            <origin rpy="0 0 ${PI / 2}" xyz="0 -0.05 -0.15"/>
-            <geometry>
-                <mesh filename="package://arduinobot_description/meshes/claw_support.STL" scale="0.01 0.01 0.01"/>
-            </geometry>
-        </visual>
-        <collision>
-            <origin rpy="0 0 ${PI / 2}" xyz="0 -0.05 -0.15"/>
-            <geometry>
-                <mesh filename="package://arduinobot_description/meshes/claw_support.STL" scale="0.01 0.01 0.01"/>
-            </geometry>
-        </collision>
-    </link>
-    <link name="gripper_right">
-        <xacro:default_inertial mass="0.01"/>
-        <visual>
-            <origin rpy="0 0 -${PI / 2}" xyz="-0.1 0.50 -0.1"/>
-            <geometry>
-                <mesh filename="package://arduinobot_description/meshes/right_finger.STL" scale="0.01 0.01 0.01"/>
-            </geometry>
-        </visual>
-        <collision>
-            <origin rpy="0 0 -${PI / 2}" xyz="-0.1 0.50 -0.1"/>
-            <geometry>
-                <mesh filename="package://arduinobot_description/meshes/right_finger.STL" scale="0.01 0.01 0.01"/>
-            </geometry>
-        </collision>
-    </link>
-    <link name="gripper_left">
-        <xacro:default_inertial mass="0.01"/>
-        <visual>
-            <origin rpy="0 0 -${PI / 2}" xyz="-0.04 0.50 -0.1"/>
-            <geometry>
-                <mesh filename="package://arduinobot_description/meshes/left_finger.STL" scale="0.01 0.01 0.01"/>
-            </geometry>
-        </visual>
-        <collision>
-            <origin rpy="0 0 -${PI / 2}" xyz="-0.04 0.50 -0.1"/>
-            <geometry>
-                <mesh filename="package://arduinobot_description/meshes/left_finger.STL" scale="0.01 0.01 0.01"/>
-            </geometry>
-        </collision>
-    </link>
-    <link name="tool_link"></link>
-    <!-- Joints -->
     <joint name="virtual_joint" type="fixed">
         <parent link="world"/>
@@ -147,54 +25,4 @@
         <origin xyz="0 0 0.307"/>
         <axis xyz="0 0 1"/>
-        <limit lower="${joint_arm_lower_limit}" upper="${joint_arm_upper_limit}"
-               effort="${effort}" velocity="${velocity}"/>
     </joint>
-    <joint name ="joint_2" type="revolute">
-        <parent link="base_plate"/>
-        <child link = "forward_drive_arm"/>
-        <origin xyz="-0.02 0 0.35"/>
-        <axis xyz="1 0 0"/>
-        <limit lower="${joint_arm_lower_limit}" upper="${joint_arm_upper_limit}"
-                effort="${effort}" velocity="${velocity}"/>
-    </joint>
-    <joint name ="joint_3" type="revolute">
-        <parent link="forward_drive_arm"/>
-        <child link = "horizontal_arm"/>
-        <origin xyz="0 0 0.8"/>
-        <axis xyz="1 0 0"/>
-        <limit lower="${joint_arm_lower_limit}" upper="${joint_arm_upper_limit}"
-               effort="${effort}" velocity="${velocity}"/>
-    </joint>
-    <joint name ="horizontal_arm_to_claw_support" type="fixed">
-        <parent link="horizontal_arm"/>
-        <child link = "claw_support"/>
-        <origin xyz="0 0.82 0"/>
-    </joint>
-    <joint name ="joint_4" type="revolute">
-        <parent link="claw_support"/>
-        <child link = "gripper_right"/>
-        <origin xyz="-0.04 0.13 -0.1"/>
-        <axis xyz="0 0 1"/>
-        <limit lower="${joint_finger_right_lower_limit}" upper="${joint_finger_right_upper_limit}"
-               effort="${effort}" velocity="${velocity}"/>
-    </joint>
-    <joint name ="joint_5" type="revolute">
-        <parent link="claw_support"/>
-        <child link = "gripper_left"/>
-        <origin xyz="-0.22 0.13 -0.1"/>
-        <axis xyz="0 0 1"/>
-        <limit lower="${joint_finger_left_lower_limit}" upper="${joint_finger_left_upper_limit}"
-               effort="${effort}" velocity="${velocity}"/>
-        <mimic joint="joint_4" multiplier="-1"/>
-    </joint>
-    <joint name ="gripper_right_to_tool" type="fixed">
-        <parent link="gripper_right"/>
-        <child link = "tool_link"/>
-        <origin xyz="0 0 0"/>
-    </joint>
-    <!-- Transmissions-->
-    <xacro:default_transmission number="1"/>
-    <xacro:default_transmission number="2"/>
-    <xacro:default_transmission number="3"/>
-    <xacro:default_transmission number="4"/>
 </robot>

Commit message: Update arduinobot.urdf.xacro

File: arduinobot_ws/src/arduinobot_description/urdf/arduinobot.urdf.xacro (robot description, xacro)
@@ -20,9 +20,3 @@
         <origin xyz="0 0 0" rpy="0 0 0"/>
     </joint>
-    <joint name ="joint_1" type="revolute">
-        <parent link="base_link"/>
-        <child link = "base_plate"/>
-        <origin xyz="0 0 0.307"/>
-        <axis xyz="0 0 1"/>
-    </joint>
 </robot>
