Commit message: uniform with lesson code

File: arduinobot_ws/src/arduinobot_description/urdf/arduinobot.urdf.xacro (robot description, xacro)
@@ -1,12 +1,12 @@
 <?xml version="1.0"?>
 <robot xmlns:xacro="http://www.ros.org/wiki/xacro" name="arduinobot">
-    <!-- Load Simulated or Real Hardware Interfaces -->
-    <xacro:arg name="is_sim" default="true"/>
-    <!-- Include XACRO Variables -->
-    <xacro:include filename="$(find arduinobot_description)/urdf/arduinobot_variables.xacro" />
     <!-- Include Gazebo Parameters -->
     <xacro:include filename="$(find arduinobot_description)/urdf/arduinobot_gazebo.xacro" />
     <!-- Include ros2_control Plugins -->
     <xacro:include filename="$(find arduinobot_description)/urdf/arduinobot_ros2_control.xacro" />
+    <!-- Useful XACRO Variables (Properties) -->
+    <xacro:property name="PI" value="3.14159265359" />
+    <xacro:property name="effort" value="30.0" />
+    <xacro:property name="velocity" value="10.0" />
     <!-- Useful Macros -->
     <xacro:macro name="default_inertial" params="mass">
@@ -23,5 +23,5 @@
             <plugin>transmission_interface/SimpleTransmission</plugin>
             <actuator name="motor_${number}" role="actuator1"/>
-            <joint name="wheel_${number}"    role="joint1">
+            <joint name="joint_${number}"    role="joint1">
                 <mechanical_reduction>1.0</mechanical_reduction>
             </joint>
@@ -135,5 +135,4 @@
         </collision>
     </link>
-    <link name="tool_link"></link>
     <!-- Joints -->
     <joint name="virtual_joint" type="fixed">
@@ -147,5 +146,5 @@
         <origin xyz="0 0 0.307"/>
         <axis xyz="0 0 1"/>
-        <limit lower="${joint_arm_lower_limit}" upper="${joint_arm_upper_limit}"
+        <limit lower="-${PI / 2}" upper="${PI / 2}"
                effort="${effort}" velocity="${velocity}"/>
     </joint>
@@ -155,5 +154,5 @@
         <origin xyz="-0.02 0 0.35"/>
         <axis xyz="1 0 0"/>
-        <limit lower="${joint_arm_lower_limit}" upper="${joint_arm_upper_limit}"
+        <limit lower="-${PI / 2}" upper="${PI / 2}"
                 effort="${effort}" velocity="${velocity}"/>
     </joint>
@@ -163,5 +162,5 @@
         <origin xyz="0 0 0.8"/>
         <axis xyz="1 0 0"/>
-        <limit lower="${joint_arm_lower_limit}" upper="${joint_arm_upper_limit}"
+        <limit lower="-${PI / 2}" upper="${PI / 2}"
                effort="${effort}" velocity="${velocity}"/>
     </joint>
@@ -176,5 +175,5 @@
         <origin xyz="-0.04 0.13 -0.1"/>
         <axis xyz="0 0 1"/>
-        <limit lower="${joint_finger_right_lower_limit}" upper="${joint_finger_right_upper_limit}"
+        <limit lower="-${PI / 2}" upper="0.0"
                effort="${effort}" velocity="${velocity}"/>
     </joint>
@@ -184,12 +183,7 @@
         <origin xyz="-0.22 0.13 -0.1"/>
         <axis xyz="0 0 1"/>
-        <limit lower="${joint_finger_left_lower_limit}" upper="${joint_finger_left_upper_limit}"
+        <limit lower="0.0" upper="${PI / 2}"
                effort="${effort}" velocity="${velocity}"/>
         <mimic joint="joint_4" multiplier="-1"/>
-    </joint>
-    <joint name ="gripper_right_to_tool" type="fixed">
-        <parent link="gripper_right"/>
-        <child link = "tool_link"/>
-        <origin xyz="0 0 0"/>
     </joint>
     <!-- Transmissions-->

File: arduinobot_ws/src/arduinobot_description/urdf/arduinobot_gazebo.xacro (robot description, xacro)
@@ -1,6 +1,4 @@
 <?xml version="1.0"?>
 <robot xmlns:xacro="http://www.ros.org/wiki/xacro" name="arduinobot">
-    <!-- Include XACRO Variables -->
-    <xacro:include filename="$(find arduinobot_description)/urdf/arduinobot_variables.xacro" />
     <!-- Gazebo ros2_control plugin -->
     <gazebo>

File: arduinobot_ws/src/arduinobot_description/urdf/arduinobot_ros2_control.xacro (robot description, xacro)
@@ -1,33 +1,14 @@
 <?xml version="1.0"?>
 <robot xmlns:xacro="http://www.ros.org/wiki/xacro" name="arduinobot">
-    <!-- Include XACRO Variables -->
-    <xacro:include filename="$(find arduinobot_description)/urdf/arduinobot_variables.xacro" />
     <ros2_control name="RobotSystem" type="system">
-    <!-- ros2_control Gazebo -->
-    <xacro:if value="$(arg is_sim)">
+        <xacro:property name="PI" value="3.14159265359" />
+        <!-- ros2_control Gazebo -->
         <hardware>
             <plugin>gazebo_ros2_control/GazeboSystem</plugin>
         </hardware>
-        <joint name="joint_5">
-            <param name="mimic">joint_4</param>
-            <param name="multiplier">-1</param>
-            <command_interface name="position">
-            <param name="min">${joint_finger_left_lower_limit}</param>
-            <param name="max">${joint_finger_left_upper_limit}</param>
-            </command_interface>
-        </joint>
-    </xacro:if>
-    <!-- ros2_control Real Robot -->
-    <xacro:unless value="$(arg is_sim)">
-        <hardware>
-          <plugin>arduinobot_controller/ArduinobotInterface</plugin>
-          <param name="port">/dev/ttyUSB0</param>
-        </hardware>
-    </xacro:unless>
-        <!-- ros2_control Common Interfaces -->
         <joint name="joint_1">
             <command_interface name="position">
-            <param name="min">${joint_arm_lower_limit}</param>
-            <param name="max">${joint_arm_upper_limit}</param>
+            <param name="min">-${PI / 2}</param>
+            <param name="max">${PI / 2}</param>
             </command_interface>
             <state_interface name="position"/>
@@ -35,6 +16,6 @@
         <joint name="joint_2">
             <command_interface name="position">
-            <param name="min">${joint_arm_lower_limit}</param>
-            <param name="max">${joint_arm_upper_limit}</param>
+            <param name="min">-${PI / 2}</param>
+            <param name="max">${PI / 2}</param>
             </command_interface>
             <state_interface name="position"/>
@@ -42,6 +23,6 @@
         <joint name="joint_3">
             <command_interface name="position">
-            <param name="min">${joint_arm_lower_limit}</param>
-            <param name="max">${joint_arm_upper_limit}</param>
+            <param name="min">-${PI / 2}</param>
+            <param name="max">${PI / 2}</param>
             </command_interface>
             <state_interface name="position"/>
@@ -49,9 +30,17 @@
         <joint name="joint_4">
             <command_interface name="position">
-            <param name="min">${joint_finger_right_lower_limit}</param>
-            <param name="max">${joint_finger_right_upper_limit}</param>
+            <param name="min">-${PI / 2}</param>
+            <param name="max">0.0</param>
             </command_interface>
             <state_interface name="position"/>
         </joint>
+        <joint name="joint_5">
+            <param name="mimic">joint_4</param>
+            <param name="multiplier">-1</param>
+            <command_interface name="position">
+            <param name="min">0.0</param>
+            <param name="max">${PI / 2}</param>
+            </command_interface>
+        </joint>
     </ros2_control>
 </robot>

Commit message: added code for last lesson

File: arduinobot_ws/src/arduinobot_description/urdf/arduinobot.urdf.xacro (robot description, xacro)
@@ -1,4 +1,6 @@
 <?xml version="1.0"?>
 <robot xmlns:xacro="http://www.ros.org/wiki/xacro" name="arduinobot">
+    <!-- Load Simulated or Real Hardware Interfaces -->
+    <xacro:arg name="is_sim" default="true"/>
     <!-- Include Gazebo Parameters -->
     <xacro:include filename="$(find arduinobot_description)/urdf/arduinobot_gazebo.xacro" />

File: arduinobot_ws/src/arduinobot_description/urdf/arduinobot_ros2_control.xacro (robot description, xacro)
@@ -2,9 +2,27 @@
 <robot xmlns:xacro="http://www.ros.org/wiki/xacro" name="arduinobot">
     <ros2_control name="RobotSystem" type="system">
-        <xacro:property name="PI" value="3.14159265359" />
-        <!-- ros2_control Gazebo -->
+    <xacro:property name="PI" value="3.14159265359" />
+    <!-- ros2_control Gazebo -->
+    <xacro:if value="$(arg is_sim)">
         <hardware>
             <plugin>gazebo_ros2_control/GazeboSystem</plugin>
         </hardware>
+        <joint name="joint_5">
+            <param name="mimic">joint_4</param>
+            <param name="multiplier">-1</param>
+            <command_interface name="position">
+            <param name="min">${joint_finger_left_lower_limit}</param>
+            <param name="max">${joint_finger_left_upper_limit}</param>
+            </command_interface>
+        </joint>
+    </xacro:if>
+    <!-- ros2_control Real Robot -->
+    <xacro:unless value="$(arg is_sim)">
+        <hardware>
+          <plugin>arduinobot_controller/ArduinobotInterface</plugin>
+          <param name="port">/dev/ttyUSB0</param>
+        </hardware>
+    </xacro:unless>
+        <!-- ros2_control Common Interfaces -->
         <joint name="joint_1">
             <command_interface name="position">
@@ -35,12 +53,4 @@
             <state_interface name="position"/>
         </joint>
-        <joint name="joint_5">
-            <param name="mimic">joint_4</param>
-            <param name="multiplier">-1</param>
-            <command_interface name="position">
-            <param name="min">0.0</param>
-            <param name="max">${PI / 2}</param>
-            </command_interface>
-        </joint>
     </ros2_control>
 </robot>

Commit message: added RGB camera

File: arduinobot_ws/src/arduinobot_description/urdf/arduinobot.urdf.xacro (robot description, xacro)
@@ -4,7 +4,7 @@
     <xacro:arg name="is_sim" default="true"/>
     <!-- Include Gazebo Parameters -->
-    <xacro:include filename="$(find arduinobot_description)/urdf/arduinobot_gazebo.xacro" />
+    <!-- <xacro:include filename="$(find arduinobot_description)/urdf/arduinobot_gazebo.xacro" /> -->
     <!-- Include ros2_control Plugins -->
-    <xacro:include filename="$(find arduinobot_description)/urdf/arduinobot_ros2_control.xacro" />
+    <!-- <xacro:include filename="$(find arduinobot_description)/urdf/arduinobot_ros2_control.xacro" /> -->
     <!-- Useful XACRO Variables (Properties) -->
     <xacro:property name="PI" value="3.14159265359" />
@@ -137,4 +137,19 @@
         </collision>
     </link>
+    <link name="rgb_camera">
+        <xacro:default_inertial mass="0.001"/>
+        <visual>
+            <origin rpy="-1.57 0 -1.57" xyz="-0.1 0.125 0.15"/>
+            <geometry>
+                <mesh filename="package://arduinobot_description/meshes/pi_camera.STL" scale="0.01 0.01 0.01"/>
+            </geometry>
+        </visual>
+        <collision>
+            <origin rpy="-1.57 0 -1.57" xyz="-0.1 0.125 0.15"/>
+            <geometry>
+                <mesh filename="package://arduinobot_description/meshes/pi_camera.STL" scale="0.01 0.01 0.01"/>
+            </geometry>
+        </collision>
+    </link>
     <!-- Joints -->
     <joint name="virtual_joint" type="fixed">
@@ -189,4 +204,9 @@
         <mimic joint="joint_4" multiplier="-1"/>
     </joint>
+    <joint name ="rgb_camera_joint" type="fixed">
+        <parent link="base_link"/>
+        <child link = "rgb_camera"/>
+        <origin xyz="0 0.45 0.2" rpy="0 -0.5 1.57"/>
+    </joint>
     <!-- Transmissions-->
     <xacro:default_transmission number="1"/>

File: arduinobot_ws/src/arduinobot_description/urdf/arduinobot_gazebo.xacro (robot description, xacro)
@@ -9,3 +9,35 @@
       </plugin>
     </gazebo>
+    <gazebo reference="rgb_camera">
+        <sensor type="camera" name="rgb_camera">
+            <always_on>true</always_on>
+            <update_rate>30.0</update_rate>
+            <camera name="rgb_camera">
+                <horizontal_fov>1.15</horizontal_fov>
+                <vertical_fov>0.71</vertical_fov>
+                <image>
+                    <width>2304</width>
+                    <height>1296</height>
+                    <format>R8G8B8</format>
+                </image>
+                <distortion>
+                    <k1>0.0</k1>
+                    <k2>0.0</k2>
+                    <k3>0.0</k3>
+                    <p1>0.0</p1>
+                    <p2>0.0</p2>
+                    <center>0.5 0.5</center>
+                </distortion>
+            </camera>
+            <plugin name="plugin_name" filename="libgazebo_ros_camera.so">
+                <ros>
+                    <remapping>~/image_raw:=image_raw</remapping>
+                    <remapping>~/camera_info:=camera_info</remapping>
+                </ros>
+                <camera_name>rgb_camera</camera_name>
+                <frame_name>rgb_camera</frame_name>
+                <hack_baseline>0.2</hack_baseline>
+            </plugin>
+        </sensor>
+      </gazebo>
 </robot>

Commit message: added support to jazzy and new gazebo

File: arduinobot_ws/src/arduinobot_description/urdf/arduinobot.urdf.xacro (robot description, xacro)
@@ -1,4 +1,6 @@
 <?xml version="1.0"?>
 <robot xmlns:xacro="http://www.ros.org/wiki/xacro" name="arduinobot">
+    <!-- Start GZ or Ignition depending on ROS 2 Version -->
+    <xacro:arg name="is_ignition" default="true"/>
     <!-- Load Simulated or Real Hardware Interfaces -->
     <xacro:arg name="is_sim" default="true"/>
@@ -21,13 +23,4 @@
         </inertial>
     </xacro:macro>
-    <xacro:macro name="default_transmission" params="number">
-        <transmission name="transmission_${number}">
-            <plugin>transmission_interface/SimpleTransmission</plugin>
-            <actuator name="motor_${number}" role="actuator1"/>
-            <joint name="joint_${number}"    role="joint1">
-                <mechanical_reduction>1.0</mechanical_reduction>
-            </joint>
-        </transmission>
-    </xacro:macro>
     <!-- Links -->
     <link name="world"/>
@@ -209,8 +202,3 @@
         <origin xyz="0 0.45 0.2" rpy="0 -0.5 1.57"/>
     </joint>
-    <!-- Transmissions-->
-    <xacro:default_transmission number="1"/>
-    <xacro:default_transmission number="2"/>
-    <xacro:default_transmission number="3"/>
-    <xacro:default_transmission number="4"/>
 </robot>

File: arduinobot_ws/src/arduinobot_description/urdf/arduinobot_gazebo.xacro (robot description, xacro)
@@ -1,43 +1,22 @@
 <?xml version="1.0"?>
 <robot xmlns:xacro="http://www.ros.org/wiki/xacro" name="arduinobot">
-    <!-- Gazebo ros2_control plugin -->
-    <gazebo>
-      <plugin filename="libgazebo_ros2_control.so" name="gazebo_ros2_control">
-        <robot_param>robot_description</robot_param>
-        <robot_param_node>robot_state_publisher</robot_param_node>
+  <!-- ROS 2 Control -->
+  <gazebo>
+    <!-- ROS 2 Humble -->
+    <xacro:if value="$(arg is_ignition)">
+      <plugin filename="ign_ros2_control-system" name="ign_ros2_control::IgnitionROS2ControlPlugin">
         <parameters>$(find arduinobot_controller)/config/arduinobot_controllers.yaml</parameters>
       </plugin>
-    </gazebo>
-    <gazebo reference="rgb_camera">
-        <sensor type="camera" name="rgb_camera">
-            <always_on>true</always_on>
-            <update_rate>30.0</update_rate>
-            <camera name="rgb_camera">
-                <horizontal_fov>1.15</horizontal_fov>
-                <vertical_fov>0.71</vertical_fov>
-                <image>
-                    <width>2304</width>
-                    <height>1296</height>
-                    <format>R8G8B8</format>
-                </image>
-                <distortion>
-                    <k1>0.0</k1>
-                    <k2>0.0</k2>
-                    <k3>0.0</k3>
-                    <p1>0.0</p1>
-                    <p2>0.0</p2>
-                    <center>0.5 0.5</center>
-                </distortion>
-            </camera>
-            <plugin name="plugin_name" filename="libgazebo_ros_camera.so">
-                <ros>
-                    <remapping>~/image_raw:=image_raw</remapping>
-                    <remapping>~/camera_info:=camera_info</remapping>
-                </ros>
-                <camera_name>rgb_camera</camera_name>
-                <frame_name>rgb_camera</frame_name>
-                <hack_baseline>0.2</hack_baseline>
-            </plugin>
-        </sensor>
-      </gazebo>
+      <plugin filename="ignition-gazebo-imu-system" name="ignition::gazebo::systems::Imu">
+      </plugin>
+    </xacro:if>
+    <!-- ROS 2 Iron or above -->
+    <xacro:unless value="$(arg is_ignition)">
+      <plugin filename="gz_ros2_control-system" name="gz_ros2_control::GazeboSimROS2ControlPlugin">
+        <parameters>$(find arduinobot_controller)/config/arduinobot_controllers.yaml</parameters>
+      </plugin>
+      <plugin filename="gz-sim-imu-system" name="gz::sim::systems::Imu">
+      </plugin>
+    </xacro:unless>
+  </gazebo>
 </robot>

File: arduinobot_ws/src/arduinobot_description/urdf/arduinobot_ros2_control.xacro (robot description, xacro)
@@ -5,7 +5,16 @@
         <!-- ros2_control Gazebo -->
         <xacro:if value="$(arg is_sim)">
-            <hardware>
-                <plugin>gazebo_ros2_control/GazeboSystem</plugin>
-            </hardware>
+            <!-- ROS 2 Humble -->
+            <xacro:if value="$(arg is_ignition)">
+                <hardware>
+                    <plugin>ign_ros2_control/IgnitionSystem</plugin>
+                </hardware>
+            </xacro:if>
+            <!-- ROS 2 Iron or above -->
+            <xacro:unless value="$(arg is_ignition)">
+                <hardware>
+                    <plugin>gz_ros2_control/GazeboSimSystem</plugin>
+                </hardware>
+            </xacro:unless>
             <joint name="joint_5">
                 <param name="mimic">joint_4</param>
@@ -24,5 +33,4 @@
             </hardware>
         </xacro:unless>
-        <!-- ros2_control Common Interfaces -->
         <joint name="joint_1">
             <command_interface name="position">
